Commit message: Fix gripper visuals and add joint sweep demo

File: rm65b_dual_arm_ws/src/rm65b_dual_arm_moveit_config/config/rm65b_dual_arm.urdf (robot description, URDF)
Before this commit: robot rm65b_dual_arm, 17 links, 16 joints
Links:
- link left_attached_scaled_gripper: geometry collision box size=0.014 0.014 0.010; collision box size=0.014 0.014 0.010
- link right_attached_scaled_gripper: geometry collision box size=0.014 0.014 0.010; collision box size=0.014 0.014 0.010
